File: hardware/_autosave-pico_logictester.kicad_sch (KiCad schematic)
At the start: 29 parts, among them J2 GPIO_5_28, J3 AKKU, J4 STEP_UP_IN, J5 5V VERSORGUNG, J6 TFT Display, Q1 AO3401A, Q2 BC547, SW1 SW_Push, U1 74HC245, U2 74HC245

Commit message: hardware: bauckup
Parts:
- J1: renamed from J?; footprint (none) -> Connector_IDC:IDC-Header_2x09_P2.54mm_Horizontal
Changed lines of the file:
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@@
 		(dnp no)
 		(fields_autoplaced yes)
-		(property "Reference" "J?"
+		(property "Reference" "J1"
 			(at 264.16 40.64 0)
 			(effects
@@
 			)
 		)
-		(property "Footprint" ""
+		(property "Footprint" "Connector_IDC:IDC-Header_2x09_P2.54mm_Horizontal"
 			(at 262.89 57.15 0)
 			(effects
@@
 			(project ""
 				(path "/ab4c5817-8853-4523-896c-e7a16e8d82cb"
-					(reference "J?")
+					(reference "J1")
 					(unit 1)
 				)
